File: kicad_files/Luna95.kicad_sch (KiCad schematic)
At the start: 22 parts

Commit message: I don't remember what I changed
Parts:
- added D? (x55): D_Small, symbol Device:D_Small
- added SW? (x55): Mechanical_Switch, symbol acheron_Symbols:Mechanical_Switch
Connections:
- new net: D?.2 (A), SW?.2 (x55)
Other:
- moved on the sheet: C?, F?, J?, R?, SW?, U?, Y?
